Commit message: Introduce links as sensor frames in URDF

File: robots/mobile_robot.urdf (robot description, URDF)
Before this commit: robot MobileRobot, 3 links, 2 joints
Links:
- added link RealSense
- added link VLP_16
Joints:
- added joint RealSenseFixedJoint: type fixed, parent Chassis, child RealSense, origin xyz=0 0 0.2 rpy=-1.57 0 -1.57
- added joint VLP_16FixedJoint: type fixed, parent Chassis, child VLP_16, origin xyz=0 0 0.2
