Commit message: Improve visual models of articulated bodies

File: robots/mobile_robot_articulated.urdf (robot description, URDF)
Before this commit: robot MobileRobot, 7 links, 6 joints
Links:
- link PanLink: geometry visual box size=0.02 0.02 0.12; visual box size=0.02 0.02 0.12
- link RealSense: geometry visual mesh filename=package:// choreonoid_ros_mobile_robot_tutorial/meshes/d435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
- link TiltLink: geometry visual cylinder length=0.02 radius=0.06
- link VLP_16: geometry visual cylinder length=0.0727 radius=0.05165
Joints:
- joint RealSenseFixedJoint: origin xyz=0 0 0 rpy=-1.57 0 -1.57 -> xyz=0 0 0.1 rpy=-1.57 0 -1.57
- joint VLP_16FixedJoint: origin (none) -> xyz=0 0 0.0287
