Commit message: Fix mobile robot models

File: model/mobile_robot_sensors.urdf (robot description, URDF)
Before this commit: robot MobileRobot, 7 links, 6 joints
Links:
- link PanLink: mass 0.1 -> 1.0; geometry visual box size=0.02 0.02 0.13; visual box size=0.02 0.02 0.13
- link RealSense: geometry visual box size=0.024 0.064 0.022; visual cylinder length=0.024 radius=0.011
- link TiltLink: mass 0.1 -> 1.0
- link VLP_16: geometry visual cylinder length=0.0717 radius=0.05165
Joints:
- joint LeftWheel: origin xyz=0 0.142 0.075 rpy=0 0 0 -> xyz=0 0.146 0.076 rpy=0 0 0
- joint PanJoint: limit lower=-3.14 upper=3.14 effort=1 velocity=1 -> (none); origin xyz=0 0 0.2 rpy=0 0 0 -> xyz=-0.02 0 0.165 rpy=0 0 0; type revolute -> continuous
- joint RealSenseFixedJoint: origin xyz=0 0 0.1 rpy=-1.57 0 -1.57 -> xyz=0.06 0 -0.02
- joint RightWheel: origin xyz=0 -0.142 0.075 rpy=0 0 0 -> xyz=0 -0.145 0.076 rpy=0 0 0
- joint TiltJoint: limit lower=-0.52 upper=0.52 effort=1 velocity=1 -> (none); origin xyz=0 0 0.1 rpy=0 0 0 -> xyz=0 0 0.12 rpy=0 0 0; type revolute -> continuous
- joint VLP_16FixedJoint: origin xyz=0 0 0.0287 -> xyz=0 0 0.04585
